File: nrf_peripheral_pcb/nrf_peripheral_pcb.kicad_sch (KiCad schematic)
At the start: 23 parts, among them U1 nRF52810-QCxx, U2 LIS2HH12, X1 32MHz

Commit message: Add pcb prices
Parts:
- BT1: Link (none) -> https://no.farnell.com/w/c/batteries-chargers/battery-holde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; Price (none) -> 2.64
- C1, C2: Link (none) -> https://no.farnell.com/multicomp/mc0603n120j500ct/cap-12pf-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; Price (none) -> 0.06
- C10, C15: Link (none) -> https://no.farnell.com/multicomp-pro/mc0603f105z100ct/cap-1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; Price (none) -> 0.062
- C11: Link (none) -> https://no.farnell.com/murata/grm188r60j106ke47d/cap-10-f-6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; Price (none) -> 0.182
- C12, C14: Link (none) -> https://no.farnell.com/yageo/cc0603zry5v8bb104/cap-0-1uf-25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; Price (none) -> 0.065
- C3: Link (none) -> https://no.farnell.com/murata/gjm1555c1hr80wb01d/cap-0-8pf-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; Price (none) -> 0.325
- C4, C5, C8: Link (none) -> https://no.farnell.com/yageo/cc0402krx5r6bb104/cap-0-1uf-10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; Price (none) -> 0.032
- C7: Link (none) -> https://no.farnell.com/multicomp/mc0402b101k500ct/cap-100pf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; Price (none) -> 0.032
- C9: Link (none) -> https://no.farnell.com/yageo/cc0603mrx5r5bb475/cap-4-7uf-6-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; Price (none) -> 0.219
- JSWD1: Price (none) -> 0
- L1: Link (none) -> https://no.farnell.com/murata/lqg15hs3n9s02d/inductor-3-9nh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; Price (none) -> 0.217
- L2: Link (none) -> https://no.farnell.com/tdk/mlz1608m100wt/inductor-10uh-20-s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; Price (none) -> 0.559
- L3: Link (none) -> https://no.farnell.com/murata/lqg15hs15nj02d/inductor-15nh-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; Price (none) -> 0.217
- R1, R2: Link (none) -> https://no.farnell.com/multicomp/mcmr06x103-jtl/res-10k-5-0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; Price (none) -> 0.031
- U1: Link (none) -> https://no.mouser.com/ProductDetail/Nordic-Semiconductor/NR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; Price (none) -> 17.76
- U2: Link (none) -> https://no.mouser.com/ProductDetail/STMicroelectronics/LIS2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; Price (none) -> 10.10
- X1: Link (none) -> https://no.farnell.com/murata/xrcgb32m000f2p00r0/crystal-32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; Price (none) -> 1.8
Changed lines of the file:
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@@
+      (effects (font (size 1.27 1.27)) hide)
+    )
+    (property "Link" "https://no.farnell.com/multicomp/mcmr06x103-jtl/res-10k-5-0-1w-0603-ceramic/dp/2073356" (id 4) (at 209.55 100.33 0)
+      (effects (font (size 1.27 1.27)) hide)
+    )
+    (property "Price" "0.031" (id 5) (at 209.55 100.33 0)
       (effects (font (size 1.27 1.27)) hide)
     )
@@
       (effects (font (size 1.27 1.27)) hide)
     )
+    (property "Link" "https://no.farnell.com/multicomp/mc0603n120j500ct/cap-12pf-50v-5-c0g-np0-0603/dp/https://no.farnell.com/multicomp/mc0402n120j500ct/cap-12pf-50v-5-c0g-np0-0402/dp/1758943" (id 4) (at 71.12 87.63 0)
+      (effects (font (size 1.27 1.27)) hide)
+    )
+    (property "Price" "0.06" (id 5) (at 71.12 87.63 0)
+      (effects (font (size 1.27 1.27)) hide)
+    )
     (pin "1")
     (pin "2")
@@
       (effects (font (size 1.27 1.27)) hide)
     )
+    (property "Link" "https://no.farnell.com/yageo/cc0603mrx5r5bb475/cap-4-7uf-6-3v-mlcc-0603/dp/3366552" (id 4) (at 127 49.53 0)
+      (effects (font (size 1.27 1.27)) hide)
+    )
+    (property "Price" "0.219" (id 5) (at 127 49.53 0)
+      (effects (font (size 1.27 1.27)) hide)
+    )
     (pin "1")
     (pin "2")
@@
       (effects (font (size 1.27 1.27)) hide)
     )
+    (property "Link" "https://no.farnell.com/tdk/mlz1608m100wt/inductor-10uh-20-shielded/dp/2215635" (id 4) (at 138.43 52.07 0)
+      (effects (font (size 1.27 1.27)) hide)
+    )
+    (property "Price" "0.559" (id 5) (at 138.43 52.07 0)
+      (effects (font (size 1.27 1.27)) hide)
+    )
     (pin "1")
     (pin "2")
@@
     )
     (property "Datasheet" "~" (id 3) (at 80.01 93.98 0)
+      (effects (font (size 1.27 1.27)) hide)
+    )
+    (property "Link" "https://no.farnell.com/murata/xrcgb32m000f2p00r0/crystal-32mhz-6pf-2-x-1-6mm/dp/2455839" (id 4) (at 80.01 93.98 0)
+      (effects (font (size 1.27 1.27)) hide)
+    )
+    (property "Price" "1.8" (id 5) (at 80.01 93.98 0)
       (effects (font (size 1.27 1.27)) hide)
     )
@@
       (effects (font (size 1.27 1.27)) hide)
     )
+    (property "Link" "https://no.farnell.com/murata/lqg15hs3n9s02d/inductor-3-9nh-0-75a-0402-multilayer/dp/2840119" (id 4) (at 97.79 74.93 0)
+      (effects (font (size 1.27 1.27)) hide)
+    )
+    (property "Price" "0.217" (id 5) (at 97.79 74.93 0)
+      (effects (font (size 1.27 1.27)) hide)
+    )
     (pin "1")
     (pin "2")
@@
       (effects (font (size 1.27 1.27)) hide)
     )
+    (property "Link" "https://no.farnell.com/murata/gjm1555c1hr80wb01d/cap-0-8pf-50v-c0g-np0-0402/dp/2781448" (id 4) (at 102.87 78.74 0)
+      (effects (font (size 1.27 1.27)) hide)
+    )
+    (property "Price" "0.325" (id 5) (at 102.87 78.74 0)
+      (effects (font (size 1.27 1.27)) hide)
+    )
     (pin "1")
     (pin "2")
@@
     )
     (property "Datasheet" "~" (id 3) (at 152.4 44.45 0)
+      (effects (font (size 1.27 1.27)) hide)
+    )
+    (property "Link" "https://no.farnell.com/multicomp-pro/mc0603f105z100ct/cap-1-f-10v-y5v-0603/dp/2629500" (id 4) (at 152.4 44.45 0)
+      (effects (font (size 1.27 1.27)) hide)
+    )
+    (property "Price" "0.062" (id 5) (at 152.4 44.45 0)
       (effects (font (size 1.27 1.27)) hide)
     )
@@
       (effects (font (size 1.27 1.27)) hide)
     )
+    (property "Link" "https://no.farnell.com/yageo/cc0603zry5v8bb104/cap-0-1uf-25v-mlcc-0603/dp/3366557" (id 4) (at 232.41 72.39 0)
+      (effects (font (size 1.27 1.27)) hide)
+    )
+    (property "Price" "0.065" (id 5) (at 232.41 72.39 0)
+      (effects (font (size 1.27 1.27)) hide)
+    )
     (pin "1")
     (pin "2")
@@
       (effects (font (size 1.27 1.27)) hide)
     )
+    (property "Price" "0" (id 4) (at 96.52 125.73 0)
+      (effects (font (size 1.27 1.27)) hide)
+    )
     (pin "1")
     (pin "2")
@@
       (effects (font (size 1.27 1.27)) hide)
     )
+    (property "Link" "https://no.farnell.com/murata/lqg15hs15nj02d/inductor-15nh-0-45a-0402-multilayer/dp/2840112" (id 4) (at 138.43 44.45 0)
+      (effects (font (size 1.27 1.27)) hide)
+    )
+    (property "Price" "0.217" (id 5) (at 138.43 44.45 0)
+      (effects (font (size 1.27 1.27)) hide)
+    )
     (pin "1")
     (pin "2")
@@
       (effects (font (size 1.27 1.27)) hide)
     )
+    (property "Link" "https://no.farnell.com/murata/grm188r60j106ke47d/cap-10-f-6-3v-10-x5r-0603/dp/2666488" (id 4) (at 222.25 72.39 0)
+      (effects (font (size 1.27 1.27)) hide)
+    )
+    (property "Price" "0.182" (id 5) (at 222.25 72.39 0)
+      (effects (font (size 1.27 1.27)) hide)
+    )
     (pin "1")
     (pin "2")
@@
     )
     (property "Datasheet" "www.st.com/resource/en/datasheet/lis2hh12.pdf" (id 3) (at 228.6 101.6 0)
+      (effects (font (size 1.27 1.27)) hide)
+    )
+    (property "Link" "https://no.mouser.com/ProductDetail/STMicroelectronics/LIS2HH12TR?qs=%2FyPOVIzmEE34aMMKbW6Cmg%3D%3D" (id 4) (at 237.49 101.6 0)
+      (effects (font (size 1.27 1.27)) hide)
+    )
+    (property "Price" "10.10" (id 5) (at 237.49 101.6 0)
       (effects (font (size 1.27 1.27)) hide)
     )
@@
     )
     (property "Datasheet" "http://infocenter.nordicsemi.com/pdf/nRF52810_PS_v1.1.pdf" (id 3) (at 120.65 87.63 0)
+      (effects (font (size 1.27 1.27)) hide)
+    )
+    (property "Link" "https://no.mouser.com/ProductDetail/Nordic-Semiconductor/NRF52810-QCAA-R7?qs=5aG0NVq1C4yRsJgd1EoNQw%3D%3D" (id 4) (at 133.35 92.71 0)
+      (effects (font (size 1.27 1.27)) hide)
+    )
+    (property "Price" "17.76" (id 5) (at 133.35 92.71 0)
       (effects (font (size 1.27 1.27)) hide)
     )
@@
       (effects (font (size 1.27 1.27)) hide)
     )
+    (property "Link" "https://no.farnell.com/multicomp/mc0603n120j500ct/cap-12pf-50v-5-c0g-np0-0603/dp/https://no.farnell.com/multicomp/mc0402n120j500ct/cap-12pf-50v-5-c0g-np0-0402/dp/1758943" (id 4) (at 71.12 99.06 0)
+      (effects (font (size 1.27 1.27)) hide)
+    )
+    (property "Price" "0.06" (id 5) (at 71.12 99.06 0)
+      (effects (font (size 1.27 1.27)) hide)
+    )
     (pin "1")
     (pin "2")
@@
       (effects (font (size 1.27 1.27)) hide)
     )
+    (property "Link" "https://no.farnell.com/yageo/cc0402krx5r6bb104/cap-0-1uf-10v-mlcc-0402/dp/3366433" (id 4) (at 138.43 29.21 0)
+      (effects (font (size 1.27 1.27)) hide)
+    )
+    (property "Price" "0.032" (id 5) (at 138.43 29.21 0)
+      (effects (font (size 1.27 1.27)) hide)
+    )
     (pin "1")
     (pin "2")
@@
       (effects (font (size 1.27 1.27)) hide)
     )
+    (property "Link" "https://no.farnell.com/yageo/cc0402krx5r6bb104/cap-0-1uf-10v-mlcc-0402/dp/3366433" (id 4) (at 152.4 29.21 0)
+      (effects (font (size 1.27 1.27)) hide)
+    )
+    (property "Price" "0.032" (id 5) (at 152.4 29.21 0)
+      (effects (font (size 1.27 1.27)) hide)
+    )
     (pin "1")
     (pin "2")
@@
     )
     (property "Datasheet" "~" (id 3) (at 109.22 49.53 0)
+      (effects (font (size 1.27 1.27)) hide)
+    )
+    (property "Link" "https://no.farnell.com/yageo/cc0402krx5r6bb104/cap-0-1uf-10v-mlcc-0402/dp/3366433" (id 4) (at 109.22 49.53 0)
+      (effects (font (size 1.27 1.27)) hide)
+    )
+    (property "Price" "0.032" (id 5) (at 109.22 49.53 0)
       (effects (font (size 1.27 1.27)) hide)
     )
@@
       (effects (font (size 1.27 1.27)) hide)
     )
+    (property "Link" "https://no.farnell.com/multicomp/mc0402b101k500ct/cap-100pf-50v-10-x7r-0402-reel/dp/2408537" (id 4) (at 72.39 49.53 0)
+      (effects (font (size 1.27 1.27)) hide)
+    )
+    (property "Price" "0.032" (id 5) (at 72.39 49.53 0)
+      (effects (font (size 1.27 1.27)) hide)
+    )
     (pin "1")
     (pin "2")
@@
       (effects (font (size 1.27 1.27)) hide)
     )
+    (property "Link" "https://no.farnell.com/w/c/batteries-chargers/battery-holders/prl/resultater?battery-sizes-accepted=2032&sort=P_PRICE" (id 4) (at 207.01 44.45 0)
+      (effects (font (size 1.27 1.27)) hide)
+    )
+    (property "Price" "2.64" (id 5) (at 207.01 44.45 0)
+      (effects (font (size 1.27 1.27)) hide)
+    )
     (pin "1")
     (pin "2")
@@
     )
     (property "Datasheet" "~" (id 3) (at 215.9 95.25 0)
+      (effects (font (size 1.27 1.27)) hide)
+    )
+    (property "Link" "https://no.farnell.com/multicomp/mcmr06x103-jtl/res-10k-5-0-1w-0603-ceramic/dp/2073356" (id 4) (at 215.9 95.25 0)
+      (effects (font (size 1.27 1.27)) hide)
+    )
+    (property "Price" "0.031" (id 5) (at 215.9 95.25 0)
       (effects (font (size 1.27 1.27)) hide)
     )
@@
       (effects (font (size 1.27 1.27)) hide)
     )
+    (property "Link" "https://no.farnell.com/multicomp-pro/mc0603f105z100ct/cap-1-f-10v-y5v-0603/dp/2629500" (id 4) (at 76.2 127 0)
+      (effects (font (size 1.27 1.27)) hide)
+    )
+    (property "Price" "0.062" (id 5) (at 76.2 127 0)
+      (effects (font (size 1.27 1.27)) hide)
+    )
     (pin "1")
     (pin "2")
@@
       (effects (font (size 1.27 1.27)) hide)
     )
+    (property "Link" "https://no.farnell.com/yageo/cc0603zry5v8bb104/cap-0-1uf-25v-mlcc-0603/dp/3366557" (id 4) (at 247.65 72.39 0)
+      (effects (font (size 1.27 1.27)) hide)
+    )
+    (property "Price" "0.065" (id 5) (at 247.65 72.39 0)
+      (effects (font (size 1.27 1.27)) hide)
+    )
